File: pcb/sabvoton-controller/sabvoton-controller.kicad_sch (KiCad schematic)
At the start: 61 parts, among them J1 CONTROLLER_HALL, J2 CONN_MAIN, J3 ENGINE_HALL, J4 DISPLAY_CONNECTOR, Q1 BSS123, Q2 BSS123, Q3 BSS123, U1 ESP32-WROOM-32, U2 XL7015E1, U3 XL7015E1, U4 NCP1117-3.3_SOT223, U5 LM1117-1.8, U6 BTS4140N, U7 LM358

Commit message: Finished PCB design
Parts:
- removed CIN4, CIN5, CIN6: C, Capacitor_SMD:C_1210_3225Metric_Pad1.33x2.70mm_HandSolder, symbol Device:C
- added CSMALL1, CSMALL10, CSMALL6, CSMALL7, CSMALL8, CSMALL9: C, Capacitor_SMD:C_1206_3216Metric, symbol Device:C
- added D3: 12V, LED_SMD:LED_1206_3216Metric, symbol Device:LED
- added D4: 5V, LED_SMD:LED_1206_3216Metric, symbol Device:LED
- added D5: 3.3V, LED_SMD:LED_1206_3216Metric, symbol Device:LED
- added D6: ESP_ON, LED_SMD:LED_1206_3216Metric, symbol Device:LED
- added R_LED_1: 600, Resistor_SMD:R_0805_2012Metric, symbol Device:R
- added R_LED_2: 130, Resistor_SMD:R_1206_3216Metric, symbol Device:R
- added R_LED_3, R_LED_4: 20, Resistor_SMD:R_1206_3216Metric, symbol Device:R
- CSMALL11, CSMALL12, CSMALL13: renamed from C?; footprint (none) -> Capacitor_SMD:C_1206_3216Metric
- J1: footprint (none) -> lib:HALL_2x6
- J2: footprint (none) -> lib:MAIN_3x10
- J3: footprint (none) -> Connector_Wire:SolderWire-0.5sqmm_1x06_P4.8mm_D0.9mm_OD2.3mm
- J4: footprint (none) -> KT_Display:SolderWire-1x4-buttons
- J5: renamed from J?; footprint (none) -> KT_Display:SolderWire-1x4-buttons
- J6, J7: renamed from J?; footprint (none) -> Connector_Wire:SolderWire-0.25sqmm_1x02_P4.2mm_D0.65mm_OD1.7mm
- J8: renamed from J?; footprint Connector_USB:USB_C_Plug_Molex_105444 -> Connector_USB:USB_Micro-B_Molex-105017-0001
- J9: renamed from J?; footprint (none) -> lib:Pogramming_1x5
- R1: value 30K -> 86K
- R10, R11, R12, R13, R14, R15, R9: renamed from R?; footprint (none) -> Resistor_SMD:R_1206_3216Metric_Pad1.30x1.75mm_HandSolder
- R5, R6, R7, R8: footprint (none) -> Resistor_SMD:R_1206_3216Metric_Pad1.30x1.75mm_HandSolder
- SW1, SW2: renamed from SW?; footprint (none) -> lib:BUTTON_SW
- U1: footprint RF_Module:ESP32-WROOM-32 -> lib:ESP32-WROOM-32
- U2: value XL7015E1 -> BUCK_12V
- U3: value XL7015E1 -> BUCK_5V
- gave numbers to parts that had none: 4
Connections:
- net 1.8V: now also U1.11 (IO26)
- net 12V: now also D3.2 (A)
- net 3.3V: now also CSMALL10.1, CSMALL6.1, CSMALL7.1, CSMALL8.1, CSMALL9.1, D5.2 (A)
- net 5V: now also D4.2 (A)
- net BATTERY_VOLTAGE: now also CSMALL1.2
- net GND: now also D1.2 (A2), D2.2 (A2), R2.2, R4.2, U2.3 (GND), U2.5 (EN), U3.3 (GND), U3.5 (EN), CSMALL1.1, CSMALL10.2, CSMALL6.2, CSMALL7.2, CSMALL8.2, CSMALL9.2, R_LED_1.2, R_LED_2.2, R_LED_3.2, R_LED_4.2; no longer CFF1.1, CFF2.1, R1.2, R2.1, R3.2, R4.1, U2.4 (FB), U3.4 (FB)
- net LED_ON: now reaches U1.30 (IO18)
- net LED_ON: now also D6.2 (A)
- new net: CFF1.1, R1.2, R2.1, U2.4 (FB)
- new net: D3.1 (K), R_LED_1.1
- new net: D6.1 (K), R_LED_4.1
- new net: D4.1 (K), R_LED_2.1
- new net: CFF2.1, R3.2, R4.1, U3.4 (FB)
- new net: D5.1 (K), R_LED_3.1
Other:
- moved on the sheet: D1, D2
